File: Lab03-STR/Exe_03/Exercicio_03.brd (EAGLE design)
At the start: 68.6 x 53.3 mm, 11 parts

Commit message: Update no projeto
Parts:
- removed D3: (no value), AUTODESK_CIRCUITS_BREADBOARD:LED5MM
- added D8: (no value), AUTODESK_CIRCUITS_BREADBOARD:LED5MM
- R1, R2, R3, R4, R5: value 1k‎Ω -> 10k‎Ω
- moved D5 25.4 mm to (5.00, 48.2)
- renumbered D4 to D7
Connections:
- removed net N$10 (its old number): R5.1, U1.2
- new net N$12: R5.1, U1.11
- new net N$8: D1.K, D2.K, D5.K, D7.K, D8.K, U1.GND.
- net N$1: now also U1.5V; no longer D1.K, D2.K, D3.K, D5.K, D7.K, U1.GND..
- net N$11: now also R4.1, U1.10; no longer R1.1, U1.11
- net N$2: now also D2.A, R1.2; no longer D1.A, R5.2
- net N$3: now also R1.1, U1.2; no longer D2.A, R4.2
- net N$4: now also D5.A, R2.2; no longer D3.A, R3.2
- net N$5: now also R2.1, U1.3; no longer D7.A, R2.2
- net N$6: now also D1.A, R3.2; no longer D5.A, R1.2
- net N$7: now also D7.A, R4.2; no longer R2.1, U1.10
- net N$9: now also D8.A, R5.2; no longer R4.1, U1.3
Changed lines of the file:
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@@
 </autorouter>
 <elements>
-<element value="" name="U1" library="AUTODESK_CIRCUITS_BREADBOARD" package="ARDUINO_UNO" x="5" y="10.08"></element><element value="" name="D1" library="AUTODESK_CIRCUITS_BREADBOARD" package="LED5MM" x="5" y="22.78"></element><element value="" name="D2" library="AUTODESK_CIRCUITS_BREADBOARD" package="LED5MM" x="5" y="35.480000000000004"></element><element value="" name="D3" library="AUTODESK_CIRCUITS_BREADBOARD" package="LED5MM" x="5" y="48.18"></element><element value="" name="D4" library="AUTODESK_CIRCUITS_BREADBOARD" package="LED5MM" x="5" y="60.879999999999995"></element><element value="" name="D5" library="AUTODESK_CIRCUITS_BREADBOARD" package="LED5MM" x="5" y="73.58"></element><element value="1k‎Ω" name="R1" library="AUTODESK_CIRCUITS_BREADBOARD" package="0207/10" x="5" y="86.28"></element><element value="1k‎Ω" name="R2" library="AUTODESK_CIRCUITS_BREADBOARD" package="0207/10" x="5" y="98.98"></element><element value="1k‎Ω" name="R3" library="AUTODESK_CIRCUITS_BREADBOARD" package="0207/10" x="5" y="111.68"></element><element value="1k‎Ω" name="R4" library="AUTODESK_CIRCUITS_BREADBOARD" package="0207/10" x="5" y="124.38000000000001"></element><element value="1k‎Ω" name="R5" library="AUTODESK_CIRCUITS_BREADBOARD" package="0207/10" x="5" y="137.08"></element></elements>
+<element value="" name="U1" library="AUTODESK_CIRCUITS_BREADBOARD" package="ARDUINO_UNO" x="5" y="10.08"></element><element value="" name="D1" library="AUTODESK_CIRCUITS_BREADBOARD" package="LED5MM" x="5" y="22.78"></element><element value="" name="D2" library="AUTODESK_CIRCUITS_BREADBOARD" package="LED5MM" x="5" y="35.480000000000004"></element><element value="" name="D5" library="AUTODESK_CIRCUITS_BREADBOARD" package="LED5MM" x="5" y="48.18"></element><element value="" name="D7" library="AUTODESK_CIRCUITS_BREADBOARD" package="LED5MM" x="5" y="60.879999999999995"></element><element value="" name="D8" library="AUTODESK_CIRCUITS_BREADBOARD" package="LED5MM" x="5" y="73.58"></element><element value="10k‎Ω" name="R1" library="AUTODESK_CIRCUITS_BREADBOARD" package="0207/10" x="5" y="86.28"></element><element value="10k‎Ω" name="R2" library="AUTODESK_CIRCUITS_BREADBOARD" package="0207/10" x="5" y="98.98"></element><element value="10k‎Ω" name="R3" library="AUTODESK_CIRCUITS_BREADBOARD" package="0207/10" x="5" y="111.68"></element><element value="10k‎Ω" name="R4" library="AUTODESK_CIRCUITS_BREADBOARD" package="0207/10" x="5" y="124.38000000000001"></element><element value="10k‎Ω" name="R5" library="AUTODESK_CIRCUITS_BREADBOARD" package="0207/10" x="5" y="137.08"></element></elements>
 <signals>
-<signal name="N$1"><contactref element="D1" pad="K"></contactref><contactref element="D2" pad="K"></contactref><wire x1="6.27" y1="22.78" x2="6.27" y2="35.480000000000004" width="0" layer="19" extent="1-1"></wire><contactref element="D3" pad="K"></contactref><wire x1="6.27" y1="35.480000000000004" x2="6.27" y2="48.18" width="0" layer="19" extent="1-1"></wire><contactref element="D4" pad="K"></contactref><wire x1="6.27" y1="48.18" x2="6.27" y2="60.879999999999995" width="0" layer="19" extent="1-1"></wire><contactref element="D5" pad="K"></contactref><wire x1="6.27" y1="60.879999999999995" x2="6.27" y2="73.58" width="0" layer="19" extent="1-1"></wire><contactref element="U1" pad="GND.."></contactref><wire x1="6.27" y1="73.58" x2="45.64" y2="12.620000000000001" width="0" layer="19" extent="1-1"></wire></signal><signal name="N$2"><contactref element="D1" pad="A"></contactref><contactref element="R5" pad="2"></contactref><wire x1="3.73" y1="22.78" x2="10.08" y2="137.08" width="0" layer="19" extent="1-1"></wire></signal><signal name="N$3"><contactref element="D2" pad="A"></contactref><contactref element="R4" pad="2"></contactref><wire x1="3.73" y1="35.480000000000004" x2="10.08" y2="124.38000000000001" width="0" layer="19" extent="1-1"></wire></signal><signal name="N$4"><contactref element="D3" pad="A"></contactref><contactref element="R3" pad="2"></contactref><wire x1="3.73" y1="48.18" x2="10.08" y2="111.68" width="0" layer="19" extent="1-1"></wire></signal><signal name="N$5"><contactref element="D4" pad="A"></contactref><contactref element="R2" pad="2"></contactref><wire x1="3.73" y1="60.879999999999995" x2="10.08" y2="98.98" width="0" layer="19" extent="1-1"></wire></signal><signal name="N$6"><contactref element="D5" pad="A"></contactref><contactref element="R1" pad="2"></contactref><wire x1="3.73" y1="73.58" x2="10.08" y2="86.28" width="0" layer="19" extent="1-1"></wire></signal><signal name="N$7"><contactref element="R2" pad="1"></contactref><contactref element="U1" pad="10"></contactref><wire x1="-0.08000000000000007" y1="98.98" x2="41.576" y2="60.879999999999995" width="0" layer="19" extent="1-1"></wire></signal><signal name="N$8"><contactref element="R3" pad="1"></contactref><contactref element="U1" pad="9"></contactref><wire x1="-0.08000000000000007" y1="111.68" x2="44.116" y2="60.879999999999995" width="0" layer="19" extent="1-1"></wire></signal><signal name="N$9"><contactref element="R4" pad="1"></contactref><contactref element="U1" pad="3"></contactref><wire x1="-0.08000000000000007" y1="124.38000000000001" x2="60.88" y2="60.879999999999995" width="0" layer="19" extent="1-1"></wire></signal><signal name="N$10"><contactref element="R5" pad="1"></contactref><contactref element="U1" pad="2"></contactref><wire x1="-0.08000000000000007" y1="137.08" x2="63.42" y2="60.879999999999995" width="0" layer="19" extent="1-1"></wire></signal><signal name="N$11"><contactref element="U1" pad="11"></contactref><contactref element="R1" pad="1"></contactref><wire x1="39.036" y1="60.879999999999995" x2="-0.08000000000000007" y2="86.28" width="0" layer="19" extent="1-1"></wire></signal></signals>
+<signal name="N$1"><contactref element="U1" pad="5V"></contactref></signal><signal name="N$2"><contactref element="R1" pad="2"></contactref><contactref element="D2" pad="A"></contactref><wire x1="10.08" y1="86.28" x2="3.73" y2="35.480000000000004" width="0" layer="19" extent="1-1"></wire></signal><signal name="N$3"><contactref element="R1" pad="1"></contactref><contactref element="U1" pad="2"></contactref><wire x1="-0.08000000000000007" y1="86.28" x2="63.42" y2="60.879999999999995" width="0" layer="19" extent="1-1"></wire></signal><signal name="N$4"><contactref element="R2" pad="2"></contactref><contactref element="D5" pad="A"></contactref><wire x1="10.08" y1="98.98" x2="3.73" y2="48.18" width="0" layer="19" extent="1-1"></wire></signal><signal name="N$5"><contactref element="R2" pad="1"></contactref><contactref element="U1" pad="3"></contactref><wire x1="-0.08000000000000007" y1="98.98" x2="60.88" y2="60.879999999999995" width="0" layer="19" extent="1-1"></wire></signal><signal name="N$6"><contactref element="D1" pad="A"></contactref><contactref element="R3" pad="2"></contactref><wire x1="3.73" y1="22.78" x2="10.08" y2="111.68" width="0" layer="19" extent="1-1"></wire></signal><signal name="N$7"><contactref element="D7" pad="A"></contactref><contactref element="R4" pad="2"></contactref><wire x1="3.73" y1="60.879999999999995" x2="10.08" y2="124.38000000000001" width="0" layer="19" extent="1-1"></wire></signal><signal name="N$8"><contactref element="D8" pad="K"></contactref><contactref element="D7" pad="K"></contactref><wire x1="6.27" y1="73.58" x2="6.27" y2="60.879999999999995" width="0" layer="19" extent="1-1"></wire><contactref element="D1" pad="K"></contactref><wire x1="6.27" y1="60.879999999999995" x2="6.27" y2="22.78" width="0" layer="19" extent="1-1"></wire><contactref element="D5" pad="K"></contactref><wire x1="6.27" y1="22.78" x2="6.27" y2="48.18" width="0" layer="19" extent="1-1"></wire><contactref element="D2" pad="K"></contactref><wire x1="6.27" y1="48.18" x2="6.27" y2="35.480000000000004" width="0" layer="19" extent="1-1"></wire><contactref element="U1" pad="GND."></contactref><wire x1="6.27" y1="35.480000000000004" x2="48.18" y2="12.620000000000001" width="0" layer="19" extent="1-1"></wire></signal><signal name="N$9"><contactref element="D8" pad="A"></contactref><contactref element="R5" pad="2"></contactref><wire x1="3.73" y1="73.58" x2="10.08" y2="137.08" width="0" layer="19" extent="1-1"></wire></signal><signal name="N$10"><contactref element="R3" pad="1"></contactref><contactref element="U1" pad="9"></contactref><wire x1="-0.08000000000000007" y1="111.68" x2="44.116" y2="60.879999999999995" width="0" layer="19" extent="1-1"></wire></signal><signal name="N$11"><contactref element="R4" pad="1"></contactref><contactref element="U1" pad="10"></contactref><wire x1="-0.08000000000000007" y1="124.38000000000001" x2="41.576" y2="60.879999999999995" width="0" layer="19" extent="1-1"></wire></signal><signal name="N$12"><contactref element="R5" pad="1"></contactref><contactref element="U1" pad="11"></contactref><wire x1="-0.08000000000000007" y1="137.08" x2="39.036" y2="60.879999999999995" width="0" layer="19" extent="1-1"></wire></signal></signals>
 </board>
 </drawing>
